File: lab1/hardware/breadboard_connections.kicad_sch (KiCad schematic)
At the start: 15 parts

Commit message: Writeup fixes during lab checkoff
Other:
- note added: "segments[0]"
- note added: "segments[1]"
- note added: "segments[2]"
- note added: "segments[3]"
- note added: "segments[4]"
- note added: "segments[5]"
- note added: "segments[6]"
Changed lines of the file:
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@@
 	)
 	(rectangle
-		(start 86.36 80.01)
+		(start 83.82 80.01)
 		(end 102.87 156.21)
 		(stroke
@@
 		(fill
 			(type none)
+		)
+	)
+	(text "segments[4]"
+		(exclude_from_sim no)
+		(at 92.456 95.504 0)
+		(effects
+			(font
+				(size 1.27 1.27)
+			)
 		)
 	)
@@
 		)
 	)
+	(text "segments[0]"
+		(exclude_from_sim no)
+		(at 91.694 133.604 0)
+		(effects
+			(font
+				(size 1.27 1.27)
+			)
+		)
+	)
 	(text "UPduino v3.1"
 		(exclude_from_sim no)
@@
 		(effects
 			(font
+				(size 1.27 1.27)
+			)
+		)
+	)
+	(text "segments[5]"
+		(exclude_from_sim no)
+		(at 92.202 146.304 0)
+		(effects
+			(font
+				(size 1.27 1.27)
+			)
+		)
+	)
+	(text "segments[1]"
+		(exclude_from_sim no)
+		(at 92.456 127.254 0)
+		(effects
+			(font
+				(size 1.27 1.27)
+			)
+		)
+	)
+	(text "segments[2]"
+		(exclude_from_sim no)
+		(at 92.456 114.554 0)
+		(effects
+			(font
+				(size 1.27 1.27)
+			)
+		)
+	)
+	(text "segments[6]"
+		(exclude_from_sim no)
+		(at 92.456 152.654 0)
+		(effects
+			(font
+				(size 1.27 1.27)
+			)
+		)
+	)
+	(text "segments[3]"
+		(exclude_from_sim no)
+		(at 92.202 101.854 0)
+		(effects
+			(font
